File: current/hardware/can.kicad_sch (KiCad schematic)
At the start: 12 parts, among them J2 2P PUSH 3.5mm, J3 2P PUSH 3.5mm, U6 TCAN3413DR

Commit message: Add Rev H RGB status and low-cost programming header
Keep sensor power and inputs unchanged. Add buffered ARGB status, nonblocking timer/DMA firmware, ordinary hand-fitted SWD header, and updated CAD/BOM/docs. Native and focused firmware checks pass. Explicitly record the canceled full power rerun as incomplete; retain full-release gates and preserve all historical packages.
Parts:
- added C74, C75: 100nF, FRC_Sensor_CAN:C_0805_2012Metric, symbol FRC_Sensor_CAN:C
- added R31: 10k, FRC_Sensor_CAN:R_0805_2012Metric, symbol FRC_Sensor_CAN:R
- added U10: SN74AHCT1G125, FRC_Sensor_CAN:SOT-23-5, symbol FRC_Sensor_CAN:LED_BUFFER
- D10: value GREEN -> SK6805-EC15; footprint FRC_Sensor_CAN:LED_0805_2012Metric -> FRC_Sensor_CAN:LED_SK6805_EC15; symbol FRC_Sensor_CAN:LED -> FRC_Sensor_CAN:RGB_LED; MPN LTST-C170KGKT -> SK6805-EC15; Notes (none) -> Single addressable RGB indicator; internal 5V, independent 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
- R30: value 1k -> 330; MPN 0805W8F1001T5E -> 0805W8F3300T5E; Notes (none) -> 330 ohm LED data series resistor; short local route after l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
Connections:
- net GND: now also D10.4 (GND), C74.2, C75.2, R31.2, U10.1 (OE_N), U10.3 (GND); no longer D10.1 (K)
- net STATUS_GREEN renamed STATUS_5V_DATA
- net STATUS_5V_DATA: now also U10.4 (Y)
- net STATUS_GREEN_A renamed STATUS_DIN
- net STATUS_DIN: now also D10.1 (DIN); no longer D10.2 (A)
- new net STATUS_DATA: R31.1, U10.2 (A)
- new net V5_INTERNAL: C74.1, C75.1, D10.2 (VDD), U10.5 (VCC)
- no-connect marks 0 -> 1
Other:
- note added: "PB3 / TIM2_CH2 drives one SK6805-EC15 through a 5 V AHCT buffer. R31 holds data LOW on reset. D10 remains powered when sensor supplies are disabled. DOUT is unused. RGB patterns are firmware diagnostics, not an independent hardware power-good indicator."
- note added: "SINGLE RGB STATUS INDICATOR / INTERNAL 5 V"
- note removed: "SINGLE STATUS INDICATOR"
- moved on the sheet: R30

Commit message: Prepare JLC-matched Rev H sourcing candidate pending simulation approval
Parts:
- R42: MPN RC1206FR-07120RL -> 1206W4F1200T5E
Changed lines of the file:
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@@
 (wire (pts (xy 142.24 99.06) (xy 149.86 99.06)) (stroke (width 0) (type default)))
 (global_label "CAN_TERM" (shape passive) (at 149.86 99.06 180) (effects (font (size 1.016 1.016)) (justify left)) (property "Intersheetrefs" "${INTERSHEET_REFS}" (at 149.86 99.06 0) (effects (font (size 1.27 1.27)) (hide yes))))
-(symbol (lib_id "FRC_Sensor_CAN:R") (at 137.16 99.06 0) (unit 1) (in_bom yes) (on_board yes) (dnp no) (property "Reference" "R42" (at 137.16 92.56 0) (effects (font (size 1.27 1.27))))(property "Value" "120" (at 137.16 95.06 0) (effects (font (size 1.016 1.016))))(property "Footprint" "FRC_Sensor_CAN:R_1206_3216Metric" (at 137.16 99.06 0) (effects (font (size 1.27 1.27)) (hide yes)))(property "Datasheet" "" (at 137.16 99.06 0) (effects (font (size 1.27 1.27)) (hide yes)))(property "MPN" "RC1206FR-07120RL" (at 137.16 99.06 0) (effects (font (size 1.27 1.27)) (hide yes)))(property "Notes" "Use termination only if board is the physical end of the CAN trunk." (at 137.16 99.06 0) (effects (font (size 1.27 1.27)) (hide yes)))(pin "1")(pin "2")(instances (project "FRC_Sensor_CAN" (path "/32fd904d-6274-5c4e-88d3-bb1b48cbb6d1/665b1307-6e60-5756-a0db-e1fad53bf5c9" (reference "R42") (unit 1)))) )
+(symbol (lib_id "FRC_Sensor_CAN:R") (at 137.16 99.06 0) (unit 1) (in_bom yes) (on_board yes) (dnp no) (property "Reference" "R42" (at 137.16 92.56 0) (effects (font (size 1.27 1.27))))(property "Value" "120" (at 137.16 95.06 0) (effects (font (size 1.016 1.016))))(property "Footprint" "FRC_Sensor_CAN:R_1206_3216Metric" (at 137.16 99.06 0) (effects (font (size 1.27 1.27)) (hide yes)))(property "Datasheet" "" (at 137.16 99.06 0) (effects (font (size 1.27 1.27)) (hide yes)))(property "MPN" "1206W4F1200T5E" (at 137.16 99.06 0) (effects (font (size 1.27 1.27)) (hide yes)))(property "Notes" "Use termination only if board is the physical end of the CAN trunk." (at 137.16 99.06 0) (effects (font (size 1.27 1.27)) (hide yes)))(pin "1")(pin "2")(instances (project "FRC_Sensor_CAN" (path "/32fd904d-6274-5c4e-88d3-bb1b48cbb6d1/665b1307-6e60-5756-a0db-e1fad53bf5c9" (reference "R42") (unit 1)))) )
 (wire (pts (xy 182.88 104.14) (xy 182.88 111.76)) (stroke (width 0) (type default)))
 (global_label "CAN_TERM" (shape passive) (at 182.88 111.76 0) (effects (font (size 1.016 1.016)) (justify right)) (property "Intersheetrefs" "${INTERSHEET_REFS}" (at 182.88 111.76 0) (effects (font (size 1.27 1.27)) (hide yes))))
