File: current/hardware/input1.kicad_sch (KiCad schematic)
At the start: 21 parts, among them J4 3P PUSH 3.5mm, Q101 AO3401A, Q102 BSS138BK, U7 LM339LV

Commit message: Rev G: protect sensor power and verify startup and fault recovery
Parts:
- U7: Notes Three digital input comparators plus protected 12V rail mon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 -> Three input comparators retained. Fourth comparator inputs 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
Changed lines of the file:
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@@
 (kicad_sch (version 20250114) (generator "eeschema") (paper "A3")
-(title_block (title "SC12 - Input 1: fixed-threshold digital input") (date "2026-09-08") (rev "F") (company "Original sensor interface design") (comment 1 "Prototype: bench validation required before robot use"))
+(title_block (title "SC12 - Input 1: fixed-threshold digital input") (date "2026-09-09") (rev "G") (company "Original sensor interface design") (comment 1 "Prototype: bench validation required before robot use"))
 (text "Input 1: fixed-threshold digital input" (at 15 15 0) (effects (font (size 2.54 2.54)) (justify left top)))
 (text "CAN-CONFIGURED INPUT BIAS / REMOVABLE SENSOR POWER" (at 15 22 0) (effects (font (size 1.7 1.7)) (justify left top)))
@@
 (symbol (lib_id "FRC_Sensor_CAN:R") (at 109.22 204.47 270) (unit 1) (in_bom yes) (on_board yes) (dnp no) (property "Reference" "R103" (at 117.22 202.97 90) (effects (font (size 1.27 1.27))))(property "Value" "20k" (at 117.22 205.97 90) (effects (font (size 1.016 1.016))))(property "Footprint" "FRC_Sensor_CAN:R_0805_2012Metric" (at 109.22 204.47 0) (effects (font (size 1.27 1.27)) (hide yes)))(property "Datasheet" "" (at 109.22 204.47 0) (effects (font (size 1.27 1.27)) (hide yes)))(property "MPN" "RC0805FR-0720KL" (at 109.22 204.47 0) (effects (font (size 1.27 1.27)) (hide yes)))(property "Notes" "" (at 109.22 204.47 0) (effects (font (size 1.27 1.27)) (hide yes)))(pin "1")(pin "2")(instances (project "FRC_Sensor_CAN" (path "/32fd904d-6274-5c4e-88d3-bb1b48cbb6d1/842f42b4-db0c-5b9a-83f5-42125535f27c" (reference "R103") (unit 1)))) )
 (symbol (lib_id "FRC_Sensor_CAN:C") (at 147.32 204.47 270) (unit 1) (in_bom yes) (on_board yes) (dnp no) (property "Reference" "C101" (at 155.32 202.97 90) (effects (font (size 1.27 1.27))))(property "Value" "1nF" (at 155.32 205.97 90) (effects (font (size 1.016 1.016))))(property "Footprint" "FRC_Sensor_CAN:C_0805_2012Metric" (at 147.32 204.47 0) (effects (font (size 1.27 1.27)) (hide yes)))(property "Datasheet" "" (at 147.32 204.47 0) (effects (font (size 1.27 1.27)) (hide yes)))(property "MPN" "CC0805JRNPO9BN102" (at 147.32 204.47 0) (effects (font (size 1.27 1.27)) (hide yes)))(property "Notes" "" (at 147.32 204.47 0) (effects (font (size 1.27 1.27)) (hide yes)))(pin "1")(pin "2")(instances (project "FRC_Sensor_CAN" (path "/32fd904d-6274-5c4e-88d3-bb1b48cbb6d1/842f42b4-db0c-5b9a-83f5-42125535f27c" (reference "C101") (unit 1)))) )
-(symbol (lib_id "FRC_Sensor_CAN:COMP4") (at 220.98 177.8 0) (unit 1) (in_bom yes) (on_board yes) (dnp no) (property "Reference" "U7" (at 220.98 168.76 0) (effects (font (size 1.27 1.27))))(property "Value" "LM339LV" (at 220.98 171.26 0) (effects (font (size 1.016 1.016))))(property "Footprint" "FRC_Sensor_CAN:SOIC-14_3.9x8.7mm_P1.27mm" (at 220.98 177.8 0) (effects (font (size 1.27 1.27)) (hide yes)))(property "Datasheet" "" (at 220.98 177.8 0) (effects (font (size 1.27 1.27)) (hide yes)))(property "MPN" "LM339LVDR" (at 220.98 177.8 0) (effects (font (size 1.27 1.27)) (hide yes)))(property "Notes" "Three digital input comparators plus protected 12V rail monitor; all four share REF_LOGIC." (at 220.98 177.8 0) (effects (font (size 1.27 1.27)) (hide yes)))(pin "5")(pin "4")(pin "2")(instances (project "FRC_Sensor_CAN" (path "/32fd904d-6274-5c4e-88d3-bb1b48cbb6d1/842f42b4-db0c-5b9a-83f5-42125535f27c" (reference "U7") (unit 1)))) )
+(symbol (lib_id "FRC_Sensor_CAN:COMP4") (at 220.98 177.8 0) (unit 1) (in_bom yes) (on_board yes) (dnp no) (property "Reference" "U7" (at 220.98 168.76 0) (effects (font (size 1.27 1.27))))(property "Value" "LM339LV" (at 220.98 171.26 0) (effects (font (size 1.016 1.016))))(property "Footprint" "FRC_Sensor_CAN:SOIC-14_3.9x8.7mm_P1.27mm" (at 220.98 177.8 0) (effects (font (size 1.27 1.27)) (hide yes)))(property "Datasheet" "" (at 220.98 177.8 0) (effects (font (size 1.27 1.27)) (hide yes)))(property "MPN" "LM339LVDR" (at 220.98 177.8 0) (effects (font (size 1.27 1.27)) (hide yes)))(property "Notes" "Three input comparators retained. Fourth comparator inputs tied to defined rails and output unconnected; rail measurements now use MCU ADC." (at 220.98 177.8 0) (effects (font (size 1.27 1.27)) (hide yes)))(pin "5")(pin "4")(pin "2")(instances (project "FRC_Sensor_CAN" (path "/32fd904d-6274-5c4e-88d3-bb1b48cbb6d1/842f42b4-db0c-5b9a-83f5-42125535f27c" (reference "U7") (unit 1)))) )
 (symbol (lib_id "FRC_Sensor_CAN:R") (at 185.42000000000002 156.21 180) (unit 1) (in_bom yes) (on_board yes) (dnp no) (property "Reference" "R104" (at 185.42 149.71 0) (effects (font (size 1.27 1.27))))(property "Value" "2.2M" (at 185.42 152.21 0) (effects (font (size 1.016 1.016))))(property "Footprint" "FRC_Sensor_CAN:R_0805_2012Metric" (at 185.42 156.21 0) (effects (font (size 1.27 1.27)) (hide yes)))(property "Datasheet" "" (at 185.42 156.21 0) (effects (font (size 1.27 1.27)) (hide yes)))(property "MPN" "RC0805FR-072M2L" (at 185.42 156.21 0) (effects (font (size 1.27 1.27)) (hide yes)))(property "Notes" "Positive feedback; fixed Schmitt thresholds with shared reference." (at 185.42 156.21 0) (effects (font (size 1.27 1.27)) (hide yes)))(pin "1")(pin "2")(instances (project "FRC_Sensor_CAN" (path "/32fd904d-6274-5c4e-88d3-bb1b48cbb6d1/842f42b4-db0c-5b9a-83f5-42125535f27c" (reference "R104") (unit 1)))) )
 (symbol (lib_id "FRC_Sensor_CAN:R") (at 281.94 163.83 270) (unit 1) (in_bom yes) (on_board yes) (dnp no) (property "Reference" "R105" (at 289.94 162.33 90) (effects (font (size 1.27 1.27))))(property "Value" "10k" (at 289.94 165.33 90) (effects (font (size 1.016 1.016))))(property "Footprint" "FRC_Sensor_CAN:R_0805_2012Metric" (at 281.94 163.83 0) (effects (font (size 1.27 1.27)) (hide yes)))(property "Datasheet" "" (at 281.94 163.83 0) (effects (font (size 1.27 1.27)) (hide yes)))(property "MPN" "0805W8F1002T5E" (at 281.94 163.83 0) (effects (font (size 1.27 1.27)) (hide yes)))(property "Notes" "" (at 281.94 163.83 0) (effects (font (size 1.27 1.27)) (hide yes)))(pin "1")(pin "2")(instances (project "FRC_Sensor_CAN" (path "/32fd904d-6274-5c4e-88d3-bb1b48cbb6d1/842f42b4-db0c-5b9a-83f5-42125535f27c" (reference "R105") (unit 1)))) )
@@
 (wire (pts (xy 292.1 255.27) (xy 292.1 262.89)) (stroke (width 0) (type default)))
 (global_label "GND" (shape passive) (at 292.1 262.89 0) (effects (font (size 1.016 1.016)) (justify right)) (property "Intersheetrefs" "${INTERSHEET_REFS}" (at 292.1 262.89 0) (effects (font (size 1.27 1.27)) (hide yes))))
-(symbol (lib_id "FRC_Sensor_CAN:COMP4") (at 292.1 247.65 0) (unit 5) (in_bom yes) (on_board yes) (dnp no) (property "Reference" "U7" (at 308.1 245.65 0) (effects (font (size 1.27 1.27))))(property "Value" "LM339LV" (at 308.1 249.65 0) (effects (font (size 1.016 1.016))))(property "Footprint" "FRC_Sensor_CAN:SOIC-14_3.9x8.7mm_P1.27mm" (at 292.1 247.65 0) (effects (font (size 1.27 1.27)) (hide yes)))(property "Datasheet" "" (at 292.1 247.65 0) (effects (font (size 1.27 1.27)) (hide yes)))(property "MPN" "LM339LVDR" (at 292.1 247.65 0) (effects (font (size 1.27 1.27)) (hide yes)))(property "Notes" "Three digital input comparators plus protected 12V rail monitor; all four share REF_LOGIC." (at 292.1 247.65 0) (effects (font (size 1.27 1.27)) (hide yes)))(pin "3")(pin "12")(instances (project "FRC_Sensor_CAN" (path "/32fd904d-6274-5c4e-88d3-bb1b48cbb6d1/842f42b4-db0c-5b9a-83f5-42125535f27c" (reference "U7") (unit 5)))) )
+(symbol (lib_id "FRC_Sensor_CAN:COMP4") (at 292.1 247.65 0) (unit 5) (in_bom yes) (on_board yes) (dnp no) (property "Reference" "U7" (at 308.1 245.65 0) (effects (font (size 1.27 1.27))))(property "Value" "LM339LV" (at 308.1 249.65 0) (effects (font (size 1.016 1.016))))(property "Footprint" "FRC_Sensor_CAN:SOIC-14_3.9x8.7mm_P1.27mm" (at 292.1 247.65 0) (effects (font (size 1.27 1.27)) (hide yes)))(property "Datasheet" "" (at 292.1 247.65 0) (effects (font (size 1.27 1.27)) (hide yes)))(property "MPN" "LM339LVDR" (at 292.1 247.65 0) (effects (font (size 1.27 1.27)) (hide yes)))(property "Notes" "Three input comparators retained. Fourth comparator inputs tied to defined rails and output unconnected; rail measurements now use MCU ADC." (at 292.1 247.65 0) (effects (font (size 1.27 1.27)) (hide yes)))(pin "3")(pin "12")(instances (project "FRC_Sensor_CAN" (path "/32fd904d-6274-5c4e-88d3-bb1b48cbb6d1/842f42b4-db0c-5b9a-83f5-42125535f27c" (reference "U7") (unit 5)))) )
 (text "0-30 V signal design range; software debounce follows the hardware filter.\nNominal thresholds near 2.0 V rising / 1.65 V falling. Final bounds are in electrical_checks.json.\nNo analog measurement, 1.8 V logic guarantee or CTRE protocol compatibility." (at 15 273 0) (effects (font (size 1.1 1.1)) (justify left top)))
 (embedded_fonts no))

Commit message: Prepare JLC-matched Rev H sourcing candidate pending simulation approval
Parts:
- R101: MPN RC0805FR-07220KL -> 0805W8F2203T5E
- R51: MPN RC0805FR-075K23L -> 0805W8F5231T5E
Changed lines of the file:
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@@
 (symbol (lib_id "FRC_Sensor_CAN:R") (at 340.36 95.25 0) (unit 1) (in_bom yes) (on_board yes) (dnp no) (property "Reference" "R109" (at 340.36 88.75 0) (effects (font (size 1.27 1.27))))(property "Value" "10k" (at 340.36 91.25 0) (effects (font (size 1.016 1.016))))(property "Footprint" "FRC_Sensor_CAN:R_1206_3216Metric" (at 340.36 95.25 0) (effects (font (size 1.27 1.27)) (hide yes)))(property "Datasheet" "" (at 340.36 95.25 0) (effects (font (size 1.27 1.27)) (hide yes)))(property "MPN" "RC1206FR-0710KL" (at 340.36 95.25 0) (effects (font (size 1.27 1.27)) (hide yes)))(property "Notes" "Electronically switched 10k pulldown; 0.09 W worst at 30 V, 1206 0.25 W." (at 340.36 95.25 0) (effects (font (size 1.27 1.27)) (hide yes)))(pin "1")(pin "2")(instances (project "FRC_Sensor_CAN" (path "/32fd904d-6274-5c4e-88d3-bb1b48cbb6d1/842f42b4-db0c-5b9a-83f5-42125535f27c" (reference "R109") (unit 1)))) )
 (text "POWER: one 2 mm cap, 1-2=5 V or 2-3=12 V; no cap=off.\nBIAS: 1k pull-up to internal 3.3 V through PMOS/diode; 10k pull-down through 60 V NMOS.\nBoth gates return OFF during reset. Software selects UP / DOWN / OFF / FLOAT / KEEPER. No bias bridges." (at 15 127 0) (effects (font (size 1.2 1.2)) (justify left top)))
-(symbol (lib_id "FRC_Sensor_CAN:R") (at 64.77 176.53 0) (unit 1) (in_bom yes) (on_board yes) (dnp no) (property "Reference" "R101" (at 64.77 170.03 0) (effects (font (size 1.27 1.27))))(property "Value" "220k" (at 64.77 172.53 0) (effects (font (size 1.016 1.016))))(property "Footprint" "FRC_Sensor_CAN:R_0805_2012Metric" (at 64.77 176.53 0) (effects (font (size 1.27 1.27)) (hide yes)))(property "Datasheet" "" (at 64.77 176.53 0) (effects (font (size 1.27 1.27)) (hide yes)))(property "MPN" "RC0805FR-07220KL" (at 64.77 176.53 0) (effects (font (size 1.27 1.27)) (hide yes)))(property "Notes" "One series resistor; loses Rev B single-resistor-short tolerance. 150 V working rating; input 0-30 V target." (at 64.77 176.53 0) (effects (font (size 1.27 1.27)) (hide yes)))(pin "1")(pin "2")(instances (project "FRC_Sensor_CAN" (path "/32fd904d-6274-5c4e-88d3-bb1b48cbb6d1/842f42b4-db0c-5b9a-83f5-42125535f27c" (reference "R101") (unit 1)))) )
+(symbol (lib_id "FRC_Sensor_CAN:R") (at 64.77 176.53 0) (unit 1) (in_bom yes) (on_board yes) (dnp no) (property "Reference" "R101" (at 64.77 170.03 0) (effects (font (size 1.27 1.27))))(property "Value" "220k" (at 64.77 172.53 0) (effects (font (size 1.016 1.016))))(property "Footprint" "FRC_Sensor_CAN:R_0805_2012Metric" (at 64.77 176.53 0) (effects (font (size 1.27 1.27)) (hide yes)))(property "Datasheet" "" (at 64.77 176.53 0) (effects (font (size 1.27 1.27)) (hide yes)))(property "MPN" "0805W8F2203T5E" (at 64.77 176.53 0) (effects (font (size 1.27 1.27)) (hide yes)))(property "Notes" "One series resistor; loses Rev B single-resistor-short tolerance. 150 V working rating; input 0-30 V target." (at 64.77 176.53 0) (effects (font (size 1.27 1.27)) (hide yes)))(pin "1")(pin "2")(instances (project "FRC_Sensor_CAN" (path "/32fd904d-6274-5c4e-88d3-bb1b48cbb6d1/842f42b4-db0c-5b9a-83f5-42125535f27c" (reference "R101") (unit 1)))) )
 (symbol (lib_id "FRC_Sensor_CAN:D") (at 25.4 201.93 90) (unit 1) (in_bom yes) (on_board yes) (dnp no) (property "Reference" "D101" (at 33.4 200.43 90) (effects (font (size 1.27 1.27))))(property "Value" "SMAJ30A" (at 33.4 203.43 90) (effects (font (size 1.016 1.016))))(property "Footprint" "FRC_Sensor_CAN:D_SMA" (at 25.4 201.93 0) (effects (font (size 1.27 1.27)) (hide yes)))(property "Datasheet" "" (at 25.4 201.93 0) (effects (font (size 1.27 1.27)) (hide yes)))(property "MPN" "SMAJ30A" (at 25.4 201.93 0) (effects (font (size 1.27 1.27)) (hide yes)))(property "Notes" "30V working standoff; unidirectional transient clamp." (at 25.4 201.93 0) (effects (font (size 1.27 1.27)) (hide yes)))(pin "2")(pin "1")(instances (project "FRC_Sensor_CAN" (path "/32fd904d-6274-5c4e-88d3-bb1b48cbb6d1/842f42b4-db0c-5b9a-83f5-42125535f27c" (reference "D101") (unit 1)))) )
 (symbol (lib_id "FRC_Sensor_CAN:R") (at 109.22 204.47 270) (unit 1) (in_bom yes) (on_board yes) (dnp no) (property "Reference" "R103" (at 117.22 202.97 90) (effects (font (size 1.27 1.27))))(property "Value" "20k" (at 117.22 205.97 90) (effects (font (size 1.016 1.016))))(property "Footprint" "FRC_Sensor_CAN:R_0805_2012Metric" (at 109.22 204.47 0) (effects (font (size 1.27 1.27)) (hide yes)))(property "Datasheet" "" (at 109.22 204.47 0) (effects (font (size 1.27 1.27)) (hide yes)))(property "MPN" "RC0805FR-0720KL" (at 109.22 204.47 0) (effects (font (size 1.27 1.27)) (hide yes)))(property "Notes" "" (at 109.22 204.47 0) (effects (font (size 1.27 1.27)) (hide yes)))(pin "1")(pin "2")(instances (project "FRC_Sensor_CAN" (path "/32fd904d-6274-5c4e-88d3-bb1b48cbb6d1/842f42b4-db0c-5b9a-83f5-42125535f27c" (reference "R103") (unit 1)))) )
@@
 (wire (pts (xy 119.38 247.65) (xy 127 247.65)) (stroke (width 0) (type default)))
 (global_label "GND" (shape passive) (at 127 247.65 180) (effects (font (size 1.016 1.016)) (justify left)) (property "Intersheetrefs" "${INTERSHEET_REFS}" (at 127 247.65 0) (effects (font (size 1.27 1.27)) (hide yes))))
-(symbol (lib_id "FRC_Sensor_CAN:R") (at 114.3 247.65 0) (unit 1) (in_bom yes) (on_board yes) (dnp no) (property "Reference" "R51" (at 114.3 241.15 0) (effects (font (size 1.27 1.27))))(property "Value" "5.23k" (at 114.3 243.65 0) (effects (font (size 1.016 1.016))))(property "Footprint" "FRC_Sensor_CAN:R_0805_2012Metric" (at 114.3 247.65 0) (effects (font (size 1.27 1.27)) (hide yes)))(property "Datasheet" "" (at 114.3 247.65 0) (effects (font (size 1.27 1.27)) (hide yes)))(property "MPN" "RC0805FR-075K23L" (at 114.3 247.65 0) (effects (font (size 1.27 1.27)) (hide yes)))(property "Notes" "" (at 114.3 247.65 0) (effects (font (size 1.27 1.27)) (hide yes)))(pin "1")(pin "2")(instances (project "FRC_Sensor_CAN" (path "/32fd904d-6274-5c4e-88d3-bb1b48cbb6d1/842f42b4-db0c-5b9a-83f5-42125535f27c" (reference "R51") (unit 1)))) )
+(symbol (lib_id "FRC_Sensor_CAN:R") (at 114.3 247.65 0) (unit 1) (in_bom yes) (on_board yes) (dnp no) (property "Reference" "R51" (at 114.3 241.15 0) (effects (font (size 1.27 1.27))))(property "Value" "5.23k" (at 114.3 243.65 0) (effects (font (size 1.016 1.016))))(property "Footprint" "FRC_Sensor_CAN:R_0805_2012Metric" (at 114.3 247.65 0) (effects (font (size 1.27 1.27)) (hide yes)))(property "Datasheet" "" (at 114.3 247.65 0) (effects (font (size 1.27 1.27)) (hide yes)))(property "MPN" "0805W8F5231T5E" (at 114.3 247.65 0) (effects (font (size 1.27 1.27)) (hide yes)))(property "Notes" "" (at 114.3 247.65 0) (effects (font (size 1.27 1.27)) (hide yes)))(pin "1")(pin "2")(instances (project "FRC_Sensor_CAN" (path "/32fd904d-6274-5c4e-88d3-bb1b48cbb6d1/842f42b4-db0c-5b9a-83f5-42125535f27c" (reference "R51") (unit 1)))) )
 (wire (pts (xy 185.42 247.65) (xy 177.8 247.65)) (stroke (width 0) (type default)))
 (global_label "REF_LOGIC" (shape passive) (at 177.8 247.65 0) (effects (font (size 1.016 1.016)) (justify right)) (property "Intersheetrefs" "${INTERSHEET_REFS}" (at 177.8 247.65 0) (effects (font (size 1.27 1.27)) (hide yes))))
