File: current/hardware/input3.kicad_sch (KiCad schematic)
At the start: 16 parts, among them J6 3P PUSH 3.5mm, Q301 AO3401A, Q302 BSS138BK, U7 LM339LV

Commit message: Rev G: protect sensor power and verify startup and fault recovery
Parts:
- U7: Notes Three digital input comparators plus protected 12V rail mon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 -> Three input comparators retained. Fourth comparator inputs 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
Changed lines of the file:
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@@
 (kicad_sch (version 20250114) (generator "eeschema") (paper "A3")
-(title_block (title "SC12 - Input 3: fixed-threshold digital input") (date "2026-09-08") (rev "F") (company "Original sensor interface design") (comment 1 "Prototype: bench validation required before robot use"))
+(title_block (title "SC12 - Input 3: fixed-threshold digital input") (date "2026-09-09") (rev "G") (company "Original sensor interface design") (comment 1 "Prototype: bench validation required before robot use"))
 (text "Input 3: fixed-threshold digital input" (at 15 15 0) (effects (font (size 2.54 2.54)) (justify left top)))
 (text "CAN-CONFIGURED INPUT BIAS / REMOVABLE SENSOR POWER" (at 15 22 0) (effects (font (size 1.7 1.7)) (justify left top)))
@@
 (symbol (lib_id "FRC_Sensor_CAN:R") (at 109.22 204.47 270) (unit 1) (in_bom yes) (on_board yes) (dnp no) (property "Reference" "R303" (at 117.22 202.97 90) (effects (font (size 1.27 1.27))))(property "Value" "20k" (at 117.22 205.97 90) (effects (font (size 1.016 1.016))))(property "Footprint" "FRC_Sensor_CAN:R_0805_2012Metric" (at 109.22 204.47 0) (effects (font (size 1.27 1.27)) (hide yes)))(property "Datasheet" "" (at 109.22 204.47 0) (effects (font (size 1.27 1.27)) (hide yes)))(property "MPN" "RC0805FR-0720KL" (at 109.22 204.47 0) (effects (font (size 1.27 1.27)) (hide yes)))(property "Notes" "" (at 109.22 204.47 0) (effects (font (size 1.27 1.27)) (hide yes)))(pin "1")(pin "2")(instances (project "FRC_Sensor_CAN" (path "/32fd904d-6274-5c4e-88d3-bb1b48cbb6d1/30a87cbd-88bf-524f-bf72-b44683ce5cbe" (reference "R303") (unit 1)))) )
 (symbol (lib_id "FRC_Sensor_CAN:C") (at 147.32 204.47 270) (unit 1) (in_bom yes) (on_board yes) (dnp no) (property "Reference" "C301" (at 155.32 202.97 90) (effects (font (size 1.27 1.27))))(property "Value" "1nF" (at 155.32 205.97 90) (effects (font (size 1.016 1.016))))(property "Footprint" "FRC_Sensor_CAN:C_0805_2012Metric" (at 147.32 204.47 0) (effects (font (size 1.27 1.27)) (hide yes)))(property "Datasheet" "" (at 147.32 204.47 0) (effects (font (size 1.27 1.27)) (hide yes)))(property "MPN" "CC0805JRNPO9BN102" (at 147.32 204.47 0) (effects (font (size 1.27 1.27)) (hide yes)))(property "Notes" "" (at 147.32 204.47 0) (effects (font (size 1.27 1.27)) (hide yes)))(pin "1")(pin "2")(instances (project "FRC_Sensor_CAN" (path "/32fd904d-6274-5c4e-88d3-bb1b48cbb6d1/30a87cbd-88bf-524f-bf72-b44683ce5cbe" (reference "C301") (unit 1)))) )
-(symbol (lib_id "FRC_Sensor_CAN:COMP4") (at 220.98 177.8 0) (unit 3) (in_bom yes) (on_board yes) (dnp no) (property "Reference" "U7" (at 220.98 168.76 0) (effects (font (size 1.27 1.27))))(property "Value" "LM339LV" (at 220.98 171.26 0) (effects (font (size 1.016 1.016))))(property "Footprint" "FRC_Sensor_CAN:SOIC-14_3.9x8.7mm_P1.27mm" (at 220.98 177.8 0) (effects (font (size 1.27 1.27)) (hide yes)))(property "Datasheet" "" (at 220.98 177.8 0) (effects (font (size 1.27 1.27)) (hide yes)))(property "MPN" "LM339LVDR" (at 220.98 177.8 0) (effects (font (size 1.27 1.27)) (hide yes)))(property "Notes" "Three digital input comparators plus protected 12V rail monitor; all four share REF_LOGIC." (at 220.98 177.8 0) (effects (font (size 1.27 1.27)) (hide yes)))(pin "9")(pin "8")(pin "14")(instances (project "FRC_Sensor_CAN" (path "/32fd904d-6274-5c4e-88d3-bb1b48cbb6d1/30a87cbd-88bf-524f-bf72-b44683ce5cbe" (reference "U7") (unit 3)))) )
+(symbol (lib_id "FRC_Sensor_CAN:COMP4") (at 220.98 177.8 0) (unit 3) (in_bom yes) (on_board yes) (dnp no) (property "Reference" "U7" (at 220.98 168.76 0) (effects (font (size 1.27 1.27))))(property "Value" "LM339LV" (at 220.98 171.26 0) (effects (font (size 1.016 1.016))))(property "Footprint" "FRC_Sensor_CAN:SOIC-14_3.9x8.7mm_P1.27mm" (at 220.98 177.8 0) (effects (font (size 1.27 1.27)) (hide yes)))(property "Datasheet" "" (at 220.98 177.8 0) (effects (font (size 1.27 1.27)) (hide yes)))(property "MPN" "LM339LVDR" (at 220.98 177.8 0) (effects (font (size 1.27 1.27)) (hide yes)))(property "Notes" "Three input comparators retained. Fourth comparator inputs tied to defined rails and output unconnected; rail measurements now use MCU ADC." (at 220.98 177.8 0) (effects (font (size 1.27 1.27)) (hide yes)))(pin "9")(pin "8")(pin "14")(instances (project "FRC_Sensor_CAN" (path "/32fd904d-6274-5c4e-88d3-bb1b48cbb6d1/30a87cbd-88bf-524f-bf72-b44683ce5cbe" (reference "U7") (unit 3)))) )
 (symbol (lib_id "FRC_Sensor_CAN:R") (at 185.42000000000002 156.21 180) (unit 1) (in_bom yes) (on_board yes) (dnp no) (property "Reference" "R304" (at 185.42 149.71 0) (effects (font (size 1.27 1.27))))(property "Value" "2.2M" (at 185.42 152.21 0) (effects (font (size 1.016 1.016))))(property "Footprint" "FRC_Sensor_CAN:R_0805_2012Metric" (at 185.42 156.21 0) (effects (font (size 1.27 1.27)) (hide yes)))(property "Datasheet" "" (at 185.42 156.21 0) (effects (font (size 1.27 1.27)) (hide yes)))(property "MPN" "RC0805FR-072M2L" (at 185.42 156.21 0) (effects (font (size 1.27 1.27)) (hide yes)))(property "Notes" "Positive feedback; fixed Schmitt thresholds with shared reference." (at 185.42 156.21 0) (effects (font (size 1.27 1.27)) (hide yes)))(pin "1")(pin "2")(instances (project "FRC_Sensor_CAN" (path "/32fd904d-6274-5c4e-88d3-bb1b48cbb6d1/30a87cbd-88bf-524f-bf72-b44683ce5cbe" (reference "R304") (unit 1)))) )
 (symbol (lib_id "FRC_Sensor_CAN:R") (at 281.94 163.83 270) (unit 1) (in_bom yes) (on_board yes) (dnp no) (property "Reference" "R305" (at 289.94 162.33 90) (effects (font (size 1.27 1.27))))(property "Value" "10k" (at 289.94 165.33 90) (effects (font (size 1.016 1.016))))(property "Footprint" "FRC_Sensor_CAN:R_0805_2012Metric" (at 281.94 163.83 0) (effects (font (size 1.27 1.27)) (hide yes)))(property "Datasheet" "" (at 281.94 163.83 0) (effects (font (size 1.27 1.27)) (hide yes)))(property "MPN" "0805W8F1002T5E" (at 281.94 163.83 0) (effects (font (size 1.27 1.27)) (hide yes)))(property "Notes" "" (at 281.94 163.83 0) (effects (font (size 1.27 1.27)) (hide yes)))(pin "1")(pin "2")(instances (project "FRC_Sensor_CAN" (path "/32fd904d-6274-5c4e-88d3-bb1b48cbb6d1/30a87cbd-88bf-524f-bf72-b44683ce5cbe" (reference "R305") (unit 1)))) )

Commit message: Prepare JLC-matched Rev H sourcing candidate pending simulation approval
Parts:
- R301: MPN RC0805FR-07220KL -> 0805W8F2203T5E
Changed lines of the file:
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@@
 (symbol (lib_id "FRC_Sensor_CAN:R") (at 340.36 95.25 0) (unit 1) (in_bom yes) (on_board yes) (dnp no) (property "Reference" "R309" (at 340.36 88.75 0) (effects (font (size 1.27 1.27))))(property "Value" "10k" (at 340.36 91.25 0) (effects (font (size 1.016 1.016))))(property "Footprint" "FRC_Sensor_CAN:R_1206_3216Metric" (at 340.36 95.25 0) (effects (font (size 1.27 1.27)) (hide yes)))(property "Datasheet" "" (at 340.36 95.25 0) (effects (font (size 1.27 1.27)) (hide yes)))(property "MPN" "RC1206FR-0710KL" (at 340.36 95.25 0) (effects (font (size 1.27 1.27)) (hide yes)))(property "Notes" "Electronically switched 10k pulldown; 0.09 W worst at 30 V, 1206 0.25 W." (at 340.36 95.25 0) (effects (font (size 1.27 1.27)) (hide yes)))(pin "1")(pin "2")(instances (project "FRC_Sensor_CAN" (path "/32fd904d-6274-5c4e-88d3-bb1b48cbb6d1/30a87cbd-88bf-524f-bf72-b44683ce5cbe" (reference "R309") (unit 1)))) )
 (text "POWER: one 2 mm cap, 1-2=5 V or 2-3=12 V; no cap=off.\nBIAS: 1k pull-up to internal 3.3 V through PMOS/diode; 10k pull-down through 60 V NMOS.\nBoth gates return OFF during reset. Software selects UP / DOWN / OFF / FLOAT / KEEPER. No bias bridges." (at 15 127 0) (effects (font (size 1.2 1.2)) (justify left top)))
-(symbol (lib_id "FRC_Sensor_CAN:R") (at 64.77 176.53 0) (unit 1) (in_bom yes) (on_board yes) (dnp no) (property "Reference" "R301" (at 64.77 170.03 0) (effects (font (size 1.27 1.27))))(property "Value" "220k" (at 64.77 172.53 0) (effects (font (size 1.016 1.016))))(property "Footprint" "FRC_Sensor_CAN:R_0805_2012Metric" (at 64.77 176.53 0) (effects (font (size 1.27 1.27)) (hide yes)))(property "Datasheet" "" (at 64.77 176.53 0) (effects (font (size 1.27 1.27)) (hide yes)))(property "MPN" "RC0805FR-07220KL" (at 64.77 176.53 0) (effects (font (size 1.27 1.27)) (hide yes)))(property "Notes" "One series resistor; loses Rev B single-resistor-short tolerance. 150 V working rating; input 0-30 V target." (at 64.77 176.53 0) (effects (font (size 1.27 1.27)) (hide yes)))(pin "1")(pin "2")(instances (project "FRC_Sensor_CAN" (path "/32fd904d-6274-5c4e-88d3-bb1b48cbb6d1/30a87cbd-88bf-524f-bf72-b44683ce5cbe" (reference "R301") (unit 1)))) )
+(symbol (lib_id "FRC_Sensor_CAN:R") (at 64.77 176.53 0) (unit 1) (in_bom yes) (on_board yes) (dnp no) (property "Reference" "R301" (at 64.77 170.03 0) (effects (font (size 1.27 1.27))))(property "Value" "220k" (at 64.77 172.53 0) (effects (font (size 1.016 1.016))))(property "Footprint" "FRC_Sensor_CAN:R_0805_2012Metric" (at 64.77 176.53 0) (effects (font (size 1.27 1.27)) (hide yes)))(property "Datasheet" "" (at 64.77 176.53 0) (effects (font (size 1.27 1.27)) (hide yes)))(property "MPN" "0805W8F2203T5E" (at 64.77 176.53 0) (effects (font (size 1.27 1.27)) (hide yes)))(property "Notes" "One series resistor; loses Rev B single-resistor-short tolerance. 150 V working rating; input 0-30 V target." (at 64.77 176.53 0) (effects (font (size 1.27 1.27)) (hide yes)))(pin "1")(pin "2")(instances (project "FRC_Sensor_CAN" (path "/32fd904d-6274-5c4e-88d3-bb1b48cbb6d1/30a87cbd-88bf-524f-bf72-b44683ce5cbe" (reference "R301") (unit 1)))) )
 (symbol (lib_id "FRC_Sensor_CAN:D") (at 25.4 201.93 90) (unit 1) (in_bom yes) (on_board yes) (dnp no) (property "Reference" "D301" (at 33.4 200.43 90) (effects (font (size 1.27 1.27))))(property "Value" "SMAJ30A" (at 33.4 203.43 90) (effects (font (size 1.016 1.016))))(property "Footprint" "FRC_Sensor_CAN:D_SMA" (at 25.4 201.93 0) (effects (font (size 1.27 1.27)) (hide yes)))(property "Datasheet" "" (at 25.4 201.93 0) (effects (font (size 1.27 1.27)) (hide yes)))(property "MPN" "SMAJ30A" (at 25.4 201.93 0) (effects (font (size 1.27 1.27)) (hide yes)))(property "Notes" "30V working standoff; unidirectional transient clamp." (at 25.4 201.93 0) (effects (font (size 1.27 1.27)) (hide yes)))(pin "2")(pin "1")(instances (project "FRC_Sensor_CAN" (path "/32fd904d-6274-5c4e-88d3-bb1b48cbb6d1/30a87cbd-88bf-524f-bf72-b44683ce5cbe" (reference "D301") (unit 1)))) )
 (symbol (lib_id "FRC_Sensor_CAN:R") (at 109.22 204.47 270) (unit 1) (in_bom yes) (on_board yes) (dnp no) (property "Reference" "R303" (at 117.22 202.97 90) (effects (font (size 1.27 1.27))))(property "Value" "20k" (at 117.22 205.97 90) (effects (font (size 1.016 1.016))))(property "Footprint" "FRC_Sensor_CAN:R_0805_2012Metric" (at 109.22 204.47 0) (effects (font (size 1.27 1.27)) (hide yes)))(property "Datasheet" "" (at 109.22 204.47 0) (effects (font (size 1.27 1.27)) (hide yes)))(property "MPN" "RC0805FR-0720KL" (at 109.22 204.47 0) (effects (font (size 1.27 1.27)) (hide yes)))(property "Notes" "" (at 109.22 204.47 0) (effects (font (size 1.27 1.27)) (hide yes)))(pin "1")(pin "2")(instances (project "FRC_Sensor_CAN" (path "/32fd904d-6274-5c4e-88d3-bb1b48cbb6d1/30a87cbd-88bf-524f-bf72-b44683ce5cbe" (reference "R303") (unit 1)))) )
