File: current/hardware/sensor_power.kicad_sch (KiCad schematic)
At the start: 4 parts, among them U4 TPS2553DBVR-1

Commit message: Rev G: protect sensor power and verify startup and fault recovery
Parts:
- added C65, C71: 1uF, FRC_Sensor_CAN:C_0805_2012Metric, symbol FRC_Sensor_CAN:C
- added C70: 47nF, FRC_Sensor_CAN:C_0805_2012Metric, symbol FRC_Sensor_CAN:C
- added D5: B240A, FRC_Sensor_CAN:D_SMA, symbol FRC_Sensor_CAN:D
- added D6: SMAJ13A, FRC_Sensor_CAN:D_SMA, symbol FRC_Sensor_CAN:D
- added Q2, Q3: BSS138BK, FRC_Sensor_CAN:SOT-23, symbol FRC_Sensor_CAN:NMOS3
- added R62: 2.61k, FRC_Sensor_CAN:R_0805_2012Metric, symbol FRC_Sensor_CAN:R
- added R68, R70: 100k, FRC_Sensor_CAN:R_0805_2012Metric, symbol FRC_Sensor_CAN:R
- added R69: 12.1k, FRC_Sensor_CAN:R_0805_2012Metric, symbol FRC_Sensor_CAN:R
- added R71, R75: 10k, FRC_Sensor_CAN:R_0805_2012Metric, symbol FRC_Sensor_CAN:R
- added U9: TPS259620DDAR, FRC_Sensor_CAN:TPS2596_DDA8, symbol FRC_Sensor_CAN:EFUSE
- U4: Notes TPS2553-1 LATCH-OFF version. Always enabled, hardware curre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 -> Independent 5 V hardware current limit; EN is MCU controlle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
Connections:
- net GND: now also C65.2, C70.2, C71.2, D5.2 (A), D6.2 (A), Q2.2 (S), Q3.2 (S), R62.2, R69.2, R71.2, R75.2, U9.1 (GND), U9.9 (EP/GND)
- net V5_INTERNAL: no longer U4.3 (EN)
- new net BOOST_12V: C65.1, D6.1 (K), R68.1, R70.1, U9.4 (IN)
- new net EFUSE_EN: Q2.3 (D), R68.2, R69.1, U9.3 (EN/UVLO)
- new net EFUSE_ILM: R62.1, U9.7 (ILM)
- new net EFUSE_INHIBIT: Q2.1 (G), Q3.3 (D), R70.2
- new net EFUSE_SS: C70.1, U9.2 (dVdt)
- new net FAULT_12V_N: U9.6 (FAULT_N)
- new net POWER_12V_EN: Q3.1 (G), R75.1
- new net POWER_5V_EN: R71.1, U4.3 (EN)
- new net SENSOR_12V: C71.1, D5.1 (K), U9.5 (OUT)
- no-connect marks 0 -> 1
Other:
- note added: "12 V BRANCH: OUTPUT ISOLATION / CONTROLLED INRUSH / HARDWARE LIMIT"
- note added: "5 V BRANCH: INDEPENDENT HARDWARE LIMIT + DEFAULT-OFF ENABLE"
- note added: "PA15 high enables 5 V. R71 holds EN low through reset and initial programming. TPS2553-1 latches off after overload; deliberate CAN service recovery cycles EN."
- note added: "U9 is after the boost reservoir: sensor shorts do not directly discharge it. R70 uses raw 12 V to inhibit U9 through Q2; PB7 HIGH enables via Q3. R75 defaults OFF without MCU power. Hardware UVLO requires about 11.1 V upstream. OVCSEL is intentionally open for the 13.8 V-class fault clamp. No reverse-powered output support. Both rails: 300 mA useful load shared between all ports; protection never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"
- note removed: "5 V sensor output: TPS2553-1 latch-off version, EN tied to input. 59k current-limit resistor. Cycle board power to clear overload. FAULT_N goes to MCU PA4, with a firmware-enabled pull-up. Design target: 300mA combined load on this rail, not per connector. Do not back-power either sensor supply output."
- note removed: "HARDWARE CURRENT LIMITING; NO FIRMWARE ENABLE"
- moved on the sheet: C11, C12, R10, U4

Commit message: Prepare JLC-matched Rev H sourcing candidate pending simulation approval
Parts:
- R10: MPN RC0805FR-0759KL -> 0805W8F5902T5E
Changed lines of the file:
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@@
 (wire (pts (xy 160.02 64.77) (xy 167.64 64.77)) (stroke (width 0) (type default)))
 (global_label "GND" (shape passive) (at 167.64 64.77 180) (effects (font (size 1.016 1.016)) (justify left)) (property "Intersheetrefs" "${INTERSHEET_REFS}" (at 167.64 64.77 0) (effects (font (size 1.27 1.27)) (hide yes))))
-(symbol (lib_id "FRC_Sensor_CAN:R") (at 154.94 64.77 0) (unit 1) (in_bom yes) (on_board yes) (dnp no) (property "Reference" "R10" (at 154.94 58.27 0) (effects (font (size 1.27 1.27))))(property "Value" "59k" (at 154.94 60.77 0) (effects (font (size 1.016 1.016))))(property "Footprint" "FRC_Sensor_CAN:R_0805_2012Metric" (at 154.94 64.77 0) (effects (font (size 1.27 1.27)) (hide yes)))(property "Datasheet" "" (at 154.94 64.77 0) (effects (font (size 1.27 1.27)) (hide yes)))(property "MPN" "RC0805FR-0759KL" (at 154.94 64.77 0) (effects (font (size 1.27 1.27)) (hide yes)))(property "Notes" "" (at 154.94 64.77 0) (effects (font (size 1.27 1.27)) (hide yes)))(pin "1")(pin "2")(instances (project "FRC_Sensor_CAN" (path "/32fd904d-6274-5c4e-88d3-bb1b48cbb6d1/0aacf9c7-060e-58ed-b759-3ac31ac433d8" (reference "R10") (unit 1)))) )
+(symbol (lib_id "FRC_Sensor_CAN:R") (at 154.94 64.77 0) (unit 1) (in_bom yes) (on_board yes) (dnp no) (property "Reference" "R10" (at 154.94 58.27 0) (effects (font (size 1.27 1.27))))(property "Value" "59k" (at 154.94 60.77 0) (effects (font (size 1.016 1.016))))(property "Footprint" "FRC_Sensor_CAN:R_0805_2012Metric" (at 154.94 64.77 0) (effects (font (size 1.27 1.27)) (hide yes)))(property "Datasheet" "" (at 154.94 64.77 0) (effects (font (size 1.27 1.27)) (hide yes)))(property "MPN" "0805W8F5902T5E" (at 154.94 64.77 0) (effects (font (size 1.27 1.27)) (hide yes)))(property "Notes" "" (at 154.94 64.77 0) (effects (font (size 1.27 1.27)) (hide yes)))(pin "1")(pin "2")(instances (project "FRC_Sensor_CAN" (path "/32fd904d-6274-5c4e-88d3-bb1b48cbb6d1/0aacf9c7-060e-58ed-b759-3ac31ac433d8" (reference "R10") (unit 1)))) )
 (wire (pts (xy 229.87 64.77) (xy 222.25 64.77)) (stroke (width 0) (type default)))
 (global_label "POWER_5V_EN" (shape passive) (at 222.25 64.77 0) (effects (font (size 1.016 1.016)) (justify right)) (property "Intersheetrefs" "${INTERSHEET_REFS}" (at 222.25 64.77 0) (effects (font (size 1.27 1.27)) (hide yes))))
