File: current/hardware/controller.kicad_sch (KiCad schematic)
At the start: 14 parts, among them J8 POGO SERVICE, U5 STM32F042K6T6, Y1 8MHz 18pF

Commit message: Rev G: protect sensor power and verify startup and fault recovery
Parts:
- C23, C24: Notes Rev F sourcing substitution: value, dielectric, voltage, to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 -> Retained sourcing substitution: value, dielectric, voltage,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
- U5: Notes Three comparator inputs PA0/1/2. PA5/6/7 active-low pull-up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 -> PA0/1/2 digital sensors; PA5/6/7 pull-up gates; PB5/PB6/PB4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
Connections:
- net BIAS_DOWN1: now also U5.28 (PB5/DOWN1); no longer U5.14 (PB0/DOWN1)
- net BIAS_DOWN2: now also U5.29 (PB6/DOWN2); no longer U5.15 (PB1/DOWN2)
- net POWER_5V_EN: now reaches U5.25 (PA15/5V_EN)
- net POWER_12V_EN: now reaches U5.30 (PB7/12V_EN)
- net PG_12V renamed FAULT_12V_N
- new net ADC_12V: U5.15 (PB1/ADC_12V)
- new net ADC_5V: U5.14 (PB0/ADC_5V)
- no-connect marks 4 -> 0
Other:
- note added: "TC2050-IDC-NL mechanical footprint; CUSTOM electrical pinout. Pin 6 is 3.3 V reference OUTPUT, never a programming power input. PB0/PB1 read sensor-rail ADCs; PA15 enables 5 V and PB7 high disables 12 V. PA3/PA4 monitor active-low fault flags. PB5/PB6/PB4 are input pull-down controls."
- note removed: "TC2050-IDC-NL mechanical footprint; CUSTOM electrical pinout. Pin 6 is 3.3 V reference OUTPUT, never a programming power input. Unused GPIOs are unconnected and initialized to analog mode. PA3 monitors 12 V PG; PA4 monitors active-low 5 V fault. No rail ADCs."

Commit message: Add Rev H RGB status and low-cost programming header
Keep sensor power and inputs unchanged. Add buffered ARGB status, nonblocking timer/DMA firmware, ordinary hand-fitted SWD header, and updated CAD/BOM/docs. Native and focused firmware checks pass. Explicitly record the canceled full power rerun as incomplete; retain full-release gates and preserve all historical packages.
Parts:
- J8: value POGO SERVICE -> 2x5 SERVICE 2.54mm; footprint FRC_Sensor_CAN:Tag-Connect_TC2050-IDC-NL_2x05_P1.27mm_Vertical -> FRC_Sensor_CAN:Service_2x05_P2.54mm; MPN (none) -> PZ254V-12-10P; Notes Standard TC2050-IDC-NL mechanical footprint; CUSTOM electri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 -> Hand-solder 2x5 2.54mm header. CUSTOM pinout; see wiring dr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; now in the parts list
Connections:
- net STATUS_GREEN renamed STATUS_DATA
Other:
- note added: "J8: hand-solder 2x5 2.54 mm header; CUSTOM electrical pinout. Pin 6 is 3.3 V reference OUTPUT, never a programming power input. PB0/PB1 read sensor-rail ADCs; PA15 enables 5 V and PB7 high enables 12 V. PA3/PA4 monitor active-low fault flags. PB5/PB6/PB4 are input pull-down controls."
- note removed: "TC2050-IDC-NL mechanical footprint; CUSTOM electrical pinout. Pin 6 is 3.3 V reference OUTPUT, never a programming power input. PB0/PB1 read sensor-rail ADCs; PA15 enables 5 V and PB7 high disables 12 V. PA3/PA4 monitor active-low fault flags. PB5/PB6/PB4 are input pull-down controls."
Changed lines of the file:
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@@
 (kicad_sch (version 20250114) (generator "eeschema") (paper "A3")
-(title_block (title "SC12 - Controller, clock, debug and status") (date "2026-09-09") (rev "G") (company "Original sensor interface design") (comment 1 "Prototype: bench validation required before robot use"))
+(title_block (title "SC12 - Controller, clock, debug and status") (date "2026-09-09") (rev "H") (company "Original sensor interface design") (comment 1 "Prototype: bench validation required before robot use"))
 (text "Controller, clock, debug and status" (at 15 15 0) (effects (font (size 2.54 2.54)) (justify left top)))
 (wire (pts (xy 67.31 78.74) (xy 59.69 78.74)) (stroke (width 0) (type default)))
@@
 (global_label "POWER_5V_EN" (shape passive) (at 130.81 106.68 180) (effects (font (size 1.016 1.016)) (justify left)) (property "Intersheetrefs" "${INTERSHEET_REFS}" (at 130.81 106.68 0) (effects (font (size 1.27 1.27)) (hide yes))))
 (wire (pts (xy 123.19 109.22) (xy 130.81 109.22)) (stroke (width 0) (type default)))
-(global_label "STATUS_GREEN" (shape passive) (at 130.81 109.22 180) (effects (font (size 1.016 1.016)) (justify left)) (property "Intersheetrefs" "${INTERSHEET_REFS}" (at 130.81 109.22 0) (effects (font (size 1.27 1.27)) (hide yes))))
+(global_label "STATUS_DATA" (shape passive) (at 130.81 109.22 180) (effects (font (size 1.016 1.016)) (justify left)) (property "Intersheetrefs" "${INTERSHEET_REFS}" (at 130.81 109.22 0) (effects (font (size 1.27 1.27)) (hide yes))))
 (symbol (lib_id "FRC_Sensor_CAN:MCU") (at 95.25 95.25 0) (unit 1) (in_bom yes) (on_board yes) (dnp no) (property "Reference" "U5" (at 95.25 64.62 0) (effects (font (size 1.27 1.27))))(property "Value" "STM32F042K6T6" (at 95.25 67.12 0) (effects (font (size 1.016 1.016))))(property "Footprint" "FRC_Sensor_CAN:LQFP-32_7x7mm_P0.8mm" (at 95.25 95.25 0) (effects (font (size 1.27 1.27)) (hide yes)))(property "Datasheet" "" (at 95.25 95.25 0) (effects (font (size 1.27 1.27)) (hide yes)))(property "MPN" "STM32F042K6T6" (at 95.25 95.25 0) (effects (font (size 1.27 1.27)) (hide yes)))(property "Notes" "PA0/1/2 digital sensors; PA5/6/7 pull-up gates; PB5/PB6/PB4 pull-down gates. PB0/PB1 measure sensor rails. PA15 enables 5V, PB7 high disables 12V. SWD/UART/CAN retained." (at 95.25 95.25 0) (effects (font (size 1.27 1.27)) (hide yes)))(pin "2")(pin "3")(pin "4")(pin "6")(pin "7")(pin "8")(pin "9")(pin "10")(pin "11")(pin "27")(pin "28")(pin "31")(pin "23")(pin "24")(pin "21")(pin "22")(pin "18")(pin "19")(pin "20")(pin "14")(pin "15")(pin "12")(pin "13")(pin "29")(pin "30")(pin "25")(pin "26")(pin "1")(pin "5")(pin "17")(pin "16")(pin "32")(instances (project "FRC_Sensor_CAN" (path "/32fd904d-6274-5c4e-88d3-bb1b48cbb6d1/019a6503-7c65-5b55-a3b1-c6260b8ca8f2" (reference "U5") (unit 1)))) )
 (wire (pts (xy 92.71 63.5) (xy 95.25 63.5)) (stroke (width 0) (type default)))
@@
 (wire (pts (xy 355.6 181.61) (xy 347.98 181.61)) (stroke (width 0) (type default)))
 (global_label "GND" (shape passive) (at 347.98 181.61 0) (effects (font (size 1.016 1.016)) (justify right)) (property "Intersheetrefs" "${INTERSHEET_REFS}" (at 347.98 181.61 0) (effects (font (size 1.27 1.27)) (hide yes))))
-(symbol (lib_id "FRC_Sensor_CAN:CONN10") (at 363.22 170.18 0) (unit 1) (in_bom no) (on_board yes) (dnp no) (property "Reference" "J8" (at 363.22 152.25 0) (effects (font (size 1.27 1.27))))(property "Value" "POGO SERVICE" (at 363.22 154.75 0) (effects (font (size 1.016 1.016))))(property "Footprint" "FRC_Sensor_CAN:Tag-Connect_TC2050-IDC-NL_2x05_P1.27mm_Vertical" (at 363.22 170.18 0) (effects (font (size 1.27 1.27)) (hide yes)))(property "Datasheet" "" (at 363.22 170.18 0) (effects (font (size 1.27 1.27)) (hide yes)))(property "MPN" "" (at 363.22 170.18 0) (effects (font (size 1.27 1.27)) (hide yes)))(property "Notes" "Standard TC2050-IDC-NL mechanical footprint; CUSTOM electrical pinout. Cable pin6 VTref output only. Follow adapter wiring table." (at 363.22 170.18 0) (effects (font (size 1.27 1.27)) (hide yes)))(pin "1")(pin "2")(pin "3")(pin "4")(pin "5")(pin "6")(pin "7")(pin "8")(pin "9")(pin "10")(instances (project "FRC_Sensor_CAN" (path "/32fd904d-6274-5c4e-88d3-bb1b48cbb6d1/019a6503-7c65-5b55-a3b1-c6260b8ca8f2" (reference "J8") (unit 1)))) )
+(symbol (lib_id "FRC_Sensor_CAN:CONN10") (at 363.22 170.18 0) (unit 1) (in_bom yes) (on_board yes) (dnp no) (property "Reference" "J8" (at 363.22 152.25 0) (effects (font (size 1.27 1.27))))(property "Value" "2x5 SERVICE 2.54mm" (at 363.22 154.75 0) (effects (font (size 1.016 1.016))))(property "Footprint" "FRC_Sensor_CAN:Service_2x05_P2.54mm" (at 363.22 170.18 0) (effects (font (size 1.27 1.27)) (hide yes)))(property "Datasheet" "" (at 363.22 170.18 0) (effects (font (size 1.27 1.27)) (hide yes)))(property "MPN" "PZ254V-12-10P" (at 363.22 170.18 0) (effects (font (size 1.27 1.27)) (hide yes)))(property "Notes" "Hand-solder 2x5 2.54mm header. CUSTOM pinout; see wiring drawing. Pin6 is target VTref sense only, never power from probe. 1.10mm finished holes." (at 363.22 170.18 0) (effects (font (size 1.27 1.27)) (hide yes)))(pin "1")(pin "2")(pin "3")(pin "4")(pin "5")(pin "6")(pin "7")(pin "8")(pin "9")(pin "10")(instances (project "FRC_Sensor_CAN" (path "/32fd904d-6274-5c4e-88d3-bb1b48cbb6d1/019a6503-7c65-5b55-a3b1-c6260b8ca8f2" (reference "J8") (unit 1)))) )
 (text "LOCAL DECOUPLING" (at 15 148 0) (effects (font (size 1.8 1.8)) (justify left top)))
 (symbol (lib_id "FRC_Sensor_CAN:C") (at 35.56 172.72 270) (unit 1) (in_bom yes) (on_board yes) (dnp no) (property "Reference" "C20" (at 43.56 171.22 90) (effects (font (size 1.27 1.27))))(property "Value" "100nF" (at 43.56 174.22 90) (effects (font (size 1.016 1.016))))(property "Footprint" "FRC_Sensor_CAN:C_0805_2012Metric" (at 35.56 172.72 0) (effects (font (size 1.27 1.27)) (hide yes)))(property "Datasheet" "" (at 35.56 172.72 0) (effects (font (size 1.27 1.27)) (hide yes)))(property "MPN" "CL21B104KCFNNNE" (at 35.56 172.72 0) (effects (font (size 1.27 1.27)) (hide yes)))(property "Notes" "" (at 35.56 172.72 0) (effects (font (size 1.27 1.27)) (hide yes)))(pin "1")(pin "2")(instances (project "FRC_Sensor_CAN" (path "/32fd904d-6274-5c4e-88d3-bb1b48cbb6d1/019a6503-7c65-5b55-a3b1-c6260b8ca8f2" (reference "C20") (unit 1)))) )
@@
 (wire (pts (xy 177.8 160.02) (xy 177.8 167.64)) (stroke (width 0) (type default)))
 (junction (at 177.8 160.02) (diameter 0) (color 0 0 0 0))
-(text "TC2050-IDC-NL mechanical footprint; CUSTOM electrical pinout.\nPin 6 is 3.3 V reference OUTPUT, never a programming power input.\nPB0/PB1 read sensor-rail ADCs; PA15 enables 5 V and PB7 high disables 12 V.\nPA3/PA4 monitor active-low fault flags. PB5/PB6/PB4 are input pull-down controls." (at 20 220 0) (effects (font (size 1.5 1.5)) (justify left top)))
+(text "J8: hand-solder 2x5 2.54 mm header; CUSTOM electrical pinout.\nPin 6 is 3.3 V reference OUTPUT, never a programming power input.\nPB0/PB1 read sensor-rail ADCs; PA15 enables 5 V and PB7 high enables 12 V.\nPA3/PA4 monitor active-low fault flags. PB5/PB6/PB4 are input pull-down controls." (at 20 220 0) (effects (font (size 1.5 1.5)) (justify left top)))
 (embedded_fonts no))

Commit message: Improve edge clearances, recess debug contacts and label wiring
Parts:
- J8: value 2x5 SERVICE 2.54mm -> 2x5 SERVICE SOCKET 2.54mm; MPN PZ254V-12-10P -> PM254V-12-10P-H85; Notes Hand-solder 2x5 2.54mm header. CUSTOM pinout; see wiring dr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 -> Hand-solder recessed female 2x5 2.54mm socket. CUSTOM pinou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
Other:
- note added: "J8: hand-solder recessed female 2x5 2.54 mm socket; CUSTOM electrical pinout. Pin 6 is 3.3 V reference OUTPUT, never a programming power input. PB0/PB1 read sensor-rail ADCs; PA15 enables 5 V and PB7 high enables 12 V. PA3/PA4 monitor active-low fault flags. PB5/PB6/PB4 are input pull-down controls."
- note removed: "J8: hand-solder 2x5 2.54 mm header; CUSTOM electrical pinout. Pin 6 is 3.3 V reference OUTPUT, never a programming power input. PB0/PB1 read sensor-rail ADCs; PA15 enables 5 V and PB7 high enables 12 V. PA3/PA4 monitor active-low fault flags. PB5/PB6/PB4 are input pull-down controls."
Changed lines of the file:
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@@
 (wire (pts (xy 355.6 181.61) (xy 347.98 181.61)) (stroke (width 0) (type default)))
 (global_label "GND" (shape passive) (at 347.98 181.61 0) (effects (font (size 1.016 1.016)) (justify right)) (property "Intersheetrefs" "${INTERSHEET_REFS}" (at 347.98 181.61 0) (effects (font (size 1.27 1.27)) (hide yes))))
-(symbol (lib_id "FRC_Sensor_CAN:CONN10") (at 363.22 170.18 0) (unit 1) (in_bom yes) (on_board yes) (dnp no) (property "Reference" "J8" (at 363.22 152.25 0) (effects (font (size 1.27 1.27))))(property "Value" "2x5 SERVICE 2.54mm" (at 363.22 154.75 0) (effects (font (size 1.016 1.016))))(property "Footprint" "FRC_Sensor_CAN:Service_2x05_P2.54mm" (at 363.22 170.18 0) (effects (font (size 1.27 1.27)) (hide yes)))(property "Datasheet" "" (at 363.22 170.18 0) (effects (font (size 1.27 1.27)) (hide yes)))(property "MPN" "PZ254V-12-10P" (at 363.22 170.18 0) (effects (font (size 1.27 1.27)) (hide yes)))(property "Notes" "Hand-solder 2x5 2.54mm header. CUSTOM pinout; see wiring drawing. Pin6 is target VTref sense only, never power from probe. 1.10mm finished holes." (at 363.22 170.18 0) (effects (font (size 1.27 1.27)) (hide yes)))(pin "1")(pin "2")(pin "3")(pin "4")(pin "5")(pin "6")(pin "7")(pin "8")(pin "9")(pin "10")(instances (project "FRC_Sensor_CAN" (path "/32fd904d-6274-5c4e-88d3-bb1b48cbb6d1/019a6503-7c65-5b55-a3b1-c6260b8ca8f2" (reference "J8") (unit 1)))) )
+(symbol (lib_id "FRC_Sensor_CAN:CONN10") (at 363.22 170.18 0) (unit 1) (in_bom yes) (on_board yes) (dnp no) (property "Reference" "J8" (at 363.22 152.25 0) (effects (font (size 1.27 1.27))))(property "Value" "2x5 SERVICE SOCKET 2.54mm" (at 363.22 154.75 0) (effects (font (size 1.016 1.016))))(property "Footprint" "FRC_Sensor_CAN:Service_2x05_P2.54mm" (at 363.22 170.18 0) (effects (font (size 1.27 1.27)) (hide yes)))(property "Datasheet" "" (at 363.22 170.18 0) (effects (font (size 1.27 1.27)) (hide yes)))(property "MPN" "PM254V-12-10P-H85" (at 363.22 170.18 0) (effects (font (size 1.27 1.27)) (hide yes)))(property "Notes" "Hand-solder recessed female 2x5 2.54mm socket. CUSTOM pinout; see wiring drawing. Pin6 is target VTref sense only, never power from probe. 1.10mm finished holes." (at 363.22 170.18 0) (effects (font (size 1.27 1.27)) (hide yes)))(pin "1")(pin "2")(pin "3")(pin "4")(pin "5")(pin "6")(pin "7")(pin "8")(pin "9")(pin "10")(instances (project "FRC_Sensor_CAN" (path "/32fd904d-6274-5c4e-88d3-bb1b48cbb6d1/019a6503-7c65-5b55-a3b1-c6260b8ca8f2" (reference "J8") (unit 1)))) )
 (text "LOCAL DECOUPLING" (at 15 148 0) (effects (font (size 1.8 1.8)) (justify left top)))
 (symbol (lib_id "FRC_Sensor_CAN:C") (at 35.56 172.72 270) (unit 1) (in_bom yes) (on_board yes) (dnp no) (property "Reference" "C20" (at 43.56 171.22 90) (effects (font (size 1.27 1.27))))(property "Value" "100nF" (at 43.56 174.22 90) (effects (font (size 1.016 1.016))))(property "Footprint" "FRC_Sensor_CAN:C_0805_2012Metric" (at 35.56 172.72 0) (effects (font (size 1.27 1.27)) (hide yes)))(property "Datasheet" "" (at 35.56 172.72 0) (effects (font (size 1.27 1.27)) (hide yes)))(property "MPN" "CL21B104KCFNNNE" (at 35.56 172.72 0) (effects (font (size 1.27 1.27)) (hide yes)))(property "Notes" "" (at 35.56 172.72 0) (effects (font (size 1.27 1.27)) (hide yes)))(pin "1")(pin "2")(instances (project "FRC_Sensor_CAN" (path "/32fd904d-6274-5c4e-88d3-bb1b48cbb6d1/019a6503-7c65-5b55-a3b1-c6260b8ca8f2" (reference "C20") (unit 1)))) )
@@
 (wire (pts (xy 177.8 160.02) (xy 177.8 167.64)) (stroke (width 0) (type default)))
 (junction (at 177.8 160.02) (diameter 0) (color 0 0 0 0))
-(text "J8: hand-solder 2x5 2.54 mm header; CUSTOM electrical pinout.\nPin 6 is 3.3 V reference OUTPUT, never a programming power input.\nPB0/PB1 read sensor-rail ADCs; PA15 enables 5 V and PB7 high enables 12 V.\nPA3/PA4 monitor active-low fault flags. PB5/PB6/PB4 are input pull-down controls." (at 20 220 0) (effects (font (size 1.5 1.5)) (justify left top)))
+(text "J8: hand-solder recessed female 2x5 2.54 mm socket; CUSTOM electrical pinout.\nPin 6 is 3.3 V reference OUTPUT, never a programming power input.\nPB0/PB1 read sensor-rail ADCs; PA15 enables 5 V and PB7 high enables 12 V.\nPA3/PA4 monitor active-low fault flags. PB5/PB6/PB4 are input pull-down controls." (at 20 220 0) (effects (font (size 1.5 1.5)) (justify left top)))
 (embedded_fonts no))

Commit message: Prepare JLC-matched Rev H sourcing candidate pending simulation approval
Parts:
- C25, C26: MPN C0805C300J5GACTU -> CC0805JRNPO9BN300
Changed lines of the file:
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@@
 (symbol (lib_id "FRC_Sensor_CAN:XTAL4") (at 251.46 58.42 0) (unit 1) (in_bom yes) (on_board yes) (dnp no) (property "Reference" "Y1" (at 251.46 51.92 0) (effects (font (size 1.27 1.27))))(property "Value" "8MHz 18pF" (at 251.46 54.42 0) (effects (font (size 1.016 1.016))))(property "Footprint" "FRC_Sensor_CAN:Abracon_ABM3B_5.0x3.2mm" (at 251.46 58.42 0) (effects (font (size 1.27 1.27)) (hide yes)))(property "Datasheet" "" (at 251.46 58.42 0) (effects (font (size 1.27 1.27)) (hide yes)))(property "MPN" "ABM3B-8.000MHZ-B2-T" (at 251.46 58.42 0) (effects (font (size 1.27 1.27)) (hide yes)))(property "Notes" "Abracon recommended land pattern: 1.8x1.2mm pads on 4.0x2.4mm centers; pads 2/4 ground." (at 251.46 58.42 0) (effects (font (size 1.27 1.27)) (hide yes)))(pin "1")(pin "3")(pin "2")(pin "4")(instances (project "FRC_Sensor_CAN" (path "/32fd904d-6274-5c4e-88d3-bb1b48cbb6d1/019a6503-7c65-5b55-a3b1-c6260b8ca8f2" (reference "Y1") (unit 1)))) )
 (symbol (lib_id "FRC_Sensor_CAN:R") (at 325.12 58.42 180) (unit 1) (in_bom yes) (on_board yes) (dnp no) (property "Reference" "R20" (at 325.12 51.92 0) (effects (font (size 1.27 1.27))))(property "Value" "0" (at 325.12 54.42 0) (effects (font (size 1.016 1.016))))(property "Footprint" "FRC_Sensor_CAN:R_0805_2012Metric" (at 325.12 58.42 0) (effects (font (size 1.27 1.27)) (hide yes)))(property "Datasheet" "" (at 325.12 58.42 0) (effects (font (size 1.27 1.27)) (hide yes)))(property "MPN" "RC0805JR-070RL" (at 325.12 58.42 0) (effects (font (size 1.27 1.27)) (hide yes)))(property "Notes" "Drive-level/startup measurement position. Tune only after oscillator characterization." (at 325.12 58.42 0) (effects (font (size 1.27 1.27)) (hide yes)))(pin "1")(pin "2")(instances (project "FRC_Sensor_CAN" (path "/32fd904d-6274-5c4e-88d3-bb1b48cbb6d1/019a6503-7c65-5b55-a3b1-c6260b8ca8f2" (reference "R20") (unit 1)))) )
-(symbol (lib_id "FRC_Sensor_CAN:C") (at 223.52 93.98 270) (unit 1) (in_bom yes) (on_board yes) (dnp no) (property "Reference" "C25" (at 231.52 92.48 90) (effects (font (size 1.27 1.27))))(property "Value" "30pF" (at 231.52 95.48 90) (effects (font (size 1.016 1.016))))(property "Footprint" "FRC_Sensor_CAN:C_0805_2012Metric" (at 223.52 93.98 0) (effects (font (size 1.27 1.27)) (hide yes)))(property "Datasheet" "" (at 223.52 93.98 0) (effects (font (size 1.27 1.27)) (hide yes)))(property "MPN" "C0805C300J5GACTU" (at 223.52 93.98 0) (effects (font (size 1.27 1.27)) (hide yes)))(property "Notes" "" (at 223.52 93.98 0) (effects (font (size 1.27 1.27)) (hide yes)))(pin "1")(pin "2")(instances (project "FRC_Sensor_CAN" (path "/32fd904d-6274-5c4e-88d3-bb1b48cbb6d1/019a6503-7c65-5b55-a3b1-c6260b8ca8f2" (reference "C25") (unit 1)))) )
-(symbol (lib_id "FRC_Sensor_CAN:C") (at 294.64 93.98 270) (unit 1) (in_bom yes) (on_board yes) (dnp no) (property "Reference" "C26" (at 302.64 92.48 90) (effects (font (size 1.27 1.27))))(property "Value" "30pF" (at 302.64 95.48 90) (effects (font (size 1.016 1.016))))(property "Footprint" "FRC_Sensor_CAN:C_0805_2012Metric" (at 294.64 93.98 0) (effects (font (size 1.27 1.27)) (hide yes)))(property "Datasheet" "" (at 294.64 93.98 0) (effects (font (size 1.27 1.27)) (hide yes)))(property "MPN" "C0805C300J5GACTU" (at 294.64 93.98 0) (effects (font (size 1.27 1.27)) (hide yes)))(property "Notes" "" (at 294.64 93.98 0) (effects (font (size 1.27 1.27)) (hide yes)))(pin "1")(pin "2")(instances (project "FRC_Sensor_CAN" (path "/32fd904d-6274-5c4e-88d3-bb1b48cbb6d1/019a6503-7c65-5b55-a3b1-c6260b8ca8f2" (reference "C26") (unit 1)))) )
+(symbol (lib_id "FRC_Sensor_CAN:C") (at 223.52 93.98 270) (unit 1) (in_bom yes) (on_board yes) (dnp no) (property "Reference" "C25" (at 231.52 92.48 90) (effects (font (size 1.27 1.27))))(property "Value" "30pF" (at 231.52 95.48 90) (effects (font (size 1.016 1.016))))(property "Footprint" "FRC_Sensor_CAN:C_0805_2012Metric" (at 223.52 93.98 0) (effects (font (size 1.27 1.27)) (hide yes)))(property "Datasheet" "" (at 223.52 93.98 0) (effects (font (size 1.27 1.27)) (hide yes)))(property "MPN" "CC0805JRNPO9BN300" (at 223.52 93.98 0) (effects (font (size 1.27 1.27)) (hide yes)))(property "Notes" "" (at 223.52 93.98 0) (effects (font (size 1.27 1.27)) (hide yes)))(pin "1")(pin "2")(instances (project "FRC_Sensor_CAN" (path "/32fd904d-6274-5c4e-88d3-bb1b48cbb6d1/019a6503-7c65-5b55-a3b1-c6260b8ca8f2" (reference "C25") (unit 1)))) )
+(symbol (lib_id "FRC_Sensor_CAN:C") (at 294.64 93.98 270) (unit 1) (in_bom yes) (on_board yes) (dnp no) (property "Reference" "C26" (at 302.64 92.48 90) (effects (font (size 1.27 1.27))))(property "Value" "30pF" (at 302.64 95.48 90) (effects (font (size 1.016 1.016))))(property "Footprint" "FRC_Sensor_CAN:C_0805_2012Metric" (at 294.64 93.98 0) (effects (font (size 1.27 1.27)) (hide yes)))(property "Datasheet" "" (at 294.64 93.98 0) (effects (font (size 1.27 1.27)) (hide yes)))(property "MPN" "CC0805JRNPO9BN300" (at 294.64 93.98 0) (effects (font (size 1.27 1.27)) (hide yes)))(property "Notes" "" (at 294.64 93.98 0) (effects (font (size 1.27 1.27)) (hide yes)))(pin "1")(pin "2")(instances (project "FRC_Sensor_CAN" (path "/32fd904d-6274-5c4e-88d3-bb1b48cbb6d1/019a6503-7c65-5b55-a3b1-c6260b8ca8f2" (reference "C26") (unit 1)))) )
 (wire (pts (xy 223.52 58.42) (xy 243.84 58.42)) (stroke (width 0) (type default)))
 (global_label "HSE_IN" (shape passive) (at 223.52 58.42 0) (effects (font (size 1.016 1.016)) (justify right)) (property "Intersheetrefs" "${INTERSHEET_REFS}" (at 223.52 58.42 0) (effects (font (size 1.27 1.27)) (hide yes))))
