File: current/hardware/controller.kicad_sch (KiCad schematic)
At the start: 14 parts, among them J8 2x5 SERVICE SOCKET 2.54mm, U5 STM32F042K6T6, Y1 8MHz 18pF

Commit message: Improve crystal startup margin and refresh pre-order verification
Parts:
- C25, C26: value 30pF -> 20pF; MPN CC0805JRNPO9BN300 -> CC0805JRNPO9BN200
Changed lines of the file:
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@@
 (symbol (lib_id "FRC_Sensor_CAN:XTAL4") (at 251.46 58.42 0) (unit 1) (in_bom yes) (on_board yes) (dnp no) (property "Reference" "Y1" (at 251.46 51.92 0) (effects (font (size 1.27 1.27))))(property "Value" "8MHz 18pF" (at 251.46 54.42 0) (effects (font (size 1.016 1.016))))(property "Footprint" "FRC_Sensor_CAN:Abracon_ABM3B_5.0x3.2mm" (at 251.46 58.42 0) (effects (font (size 1.27 1.27)) (hide yes)))(property "Datasheet" "" (at 251.46 58.42 0) (effects (font (size 1.27 1.27)) (hide yes)))(property "MPN" "ABM3B-8.000MHZ-B2-T" (at 251.46 58.42 0) (effects (font (size 1.27 1.27)) (hide yes)))(property "Notes" "Abracon recommended land pattern: 1.8x1.2mm pads on 4.0x2.4mm centers; pads 2/4 ground." (at 251.46 58.42 0) (effects (font (size 1.27 1.27)) (hide yes)))(pin "1")(pin "3")(pin "2")(pin "4")(instances (project "FRC_Sensor_CAN" (path "/32fd904d-6274-5c4e-88d3-bb1b48cbb6d1/019a6503-7c65-5b55-a3b1-c6260b8ca8f2" (reference "Y1") (unit 1)))) )
 (symbol (lib_id "FRC_Sensor_CAN:R") (at 325.12 58.42 180) (unit 1) (in_bom yes) (on_board yes) (dnp no) (property "Reference" "R20" (at 325.12 51.92 0) (effects (font (size 1.27 1.27))))(property "Value" "0" (at 325.12 54.42 0) (effects (font (size 1.016 1.016))))(property "Footprint" "FRC_Sensor_CAN:R_0805_2012Metric" (at 325.12 58.42 0) (effects (font (size 1.27 1.27)) (hide yes)))(property "Datasheet" "" (at 325.12 58.42 0) (effects (font (size 1.27 1.27)) (hide yes)))(property "MPN" "RC0805JR-070RL" (at 325.12 58.42 0) (effects (font (size 1.27 1.27)) (hide yes)))(property "Notes" "Drive-level/startup measurement position. Tune only after oscillator characterization." (at 325.12 58.42 0) (effects (font (size 1.27 1.27)) (hide yes)))(pin "1")(pin "2")(instances (project "FRC_Sensor_CAN" (path "/32fd904d-6274-5c4e-88d3-bb1b48cbb6d1/019a6503-7c65-5b55-a3b1-c6260b8ca8f2" (reference "R20") (unit 1)))) )
-(symbol (lib_id "FRC_Sensor_CAN:C") (at 223.52 93.98 270) (unit 1) (in_bom yes) (on_board yes) (dnp no) (property "Reference" "C25" (at 231.52 92.48 90) (effects (font (size 1.27 1.27))))(property "Value" "30pF" (at 231.52 95.48 90) (effects (font (size 1.016 1.016))))(property "Footprint" "FRC_Sensor_CAN:C_0805_2012Metric" (at 223.52 93.98 0) (effects (font (size 1.27 1.27)) (hide yes)))(property "Datasheet" "" (at 223.52 93.98 0) (effects (font (size 1.27 1.27)) (hide yes)))(property "MPN" "CC0805JRNPO9BN300" (at 223.52 93.98 0) (effects (font (size 1.27 1.27)) (hide yes)))(property "Notes" "" (at 223.52 93.98 0) (effects (font (size 1.27 1.27)) (hide yes)))(pin "1")(pin "2")(instances (project "FRC_Sensor_CAN" (path "/32fd904d-6274-5c4e-88d3-bb1b48cbb6d1/019a6503-7c65-5b55-a3b1-c6260b8ca8f2" (reference "C25") (unit 1)))) )
-(symbol (lib_id "FRC_Sensor_CAN:C") (at 294.64 93.98 270) (unit 1) (in_bom yes) (on_board yes) (dnp no) (property "Reference" "C26" (at 302.64 92.48 90) (effects (font (size 1.27 1.27))))(property "Value" "30pF" (at 302.64 95.48 90) (effects (font (size 1.016 1.016))))(property "Footprint" "FRC_Sensor_CAN:C_0805_2012Metric" (at 294.64 93.98 0) (effects (font (size 1.27 1.27)) (hide yes)))(property "Datasheet" "" (at 294.64 93.98 0) (effects (font (size 1.27 1.27)) (hide yes)))(property "MPN" "CC0805JRNPO9BN300" (at 294.64 93.98 0) (effects (font (size 1.27 1.27)) (hide yes)))(property "Notes" "" (at 294.64 93.98 0) (effects (font (size 1.27 1.27)) (hide yes)))(pin "1")(pin "2")(instances (project "FRC_Sensor_CAN" (path "/32fd904d-6274-5c4e-88d3-bb1b48cbb6d1/019a6503-7c65-5b55-a3b1-c6260b8ca8f2" (reference "C26") (unit 1)))) )
+(symbol (lib_id "FRC_Sensor_CAN:C") (at 223.52 93.98 270) (unit 1) (in_bom yes) (on_board yes) (dnp no) (property "Reference" "C25" (at 231.52 92.48 90) (effects (font (size 1.27 1.27))))(property "Value" "20pF" (at 231.52 95.48 90) (effects (font (size 1.016 1.016))))(property "Footprint" "FRC_Sensor_CAN:C_0805_2012Metric" (at 223.52 93.98 0) (effects (font (size 1.27 1.27)) (hide yes)))(property "Datasheet" "" (at 223.52 93.98 0) (effects (font (size 1.27 1.27)) (hide yes)))(property "MPN" "CC0805JRNPO9BN200" (at 223.52 93.98 0) (effects (font (size 1.27 1.27)) (hide yes)))(property "Notes" "" (at 223.52 93.98 0) (effects (font (size 1.27 1.27)) (hide yes)))(pin "1")(pin "2")(instances (project "FRC_Sensor_CAN" (path "/32fd904d-6274-5c4e-88d3-bb1b48cbb6d1/019a6503-7c65-5b55-a3b1-c6260b8ca8f2" (reference "C25") (unit 1)))) )
+(symbol (lib_id "FRC_Sensor_CAN:C") (at 294.64 93.98 270) (unit 1) (in_bom yes) (on_board yes) (dnp no) (property "Reference" "C26" (at 302.64 92.48 90) (effects (font (size 1.27 1.27))))(property "Value" "20pF" (at 302.64 95.48 90) (effects (font (size 1.016 1.016))))(property "Footprint" "FRC_Sensor_CAN:C_0805_2012Metric" (at 294.64 93.98 0) (effects (font (size 1.27 1.27)) (hide yes)))(property "Datasheet" "" (at 294.64 93.98 0) (effects (font (size 1.27 1.27)) (hide yes)))(property "MPN" "CC0805JRNPO9BN200" (at 294.64 93.98 0) (effects (font (size 1.27 1.27)) (hide yes)))(property "Notes" "" (at 294.64 93.98 0) (effects (font (size 1.27 1.27)) (hide yes)))(pin "1")(pin "2")(instances (project "FRC_Sensor_CAN" (path "/32fd904d-6274-5c4e-88d3-bb1b48cbb6d1/019a6503-7c65-5b55-a3b1-c6260b8ca8f2" (reference "C26") (unit 1)))) )
 (wire (pts (xy 223.52 58.42) (xy 243.84 58.42)) (stroke (width 0) (type default)))
 (global_label "HSE_IN" (shape passive) (at 223.52 58.42 0) (effects (font (size 1.016 1.016)) (justify right)) (property "Intersheetrefs" "${INTERSHEET_REFS}" (at 223.52 58.42 0) (effects (font (size 1.27 1.27)) (hide yes))))
